Commit message: final robot

File: urdf/coke_can.urdf (robot description, URDF)
Before this commit: robot coke, 1 links, 0 joints
Links:
- link tin: geometry collision cylinder length=0.5 radius=0.09; visual cylinder length=0.5 radius=0.09

File: urdf/my_robot.urdf (robot description, URDF)
Before this commit: robot gripper_robot, 9 links, 8 joints
Links:
- link camera_link: geometry collision box size=0.1 0.1 0.1; visual box size=0.1 0.1 0.1
- link link5: geometry collision box size=0.2 0.1 0.7; visual box size=0.2 0.1 0.7
- link link6: geometry collision box size=0.2 0.05 0.7; visual box size=0.2 0.1 0.7
Joints:
- joint camera_joint: origin xyz=0.15 0 -0.1 rpy=0 -1.5708 0 -> xyz=-0.15 0 0.1 rpy=0 -1.5708 0
- joint joint5: limit lower=-0.16 upper=0.0 effort=50 velocity=100 -> lower=-0.3 upper=0.0 effort=50 velocity=100
- joint joint6: limit lower=0.0 upper=0.16 effort=50 velocity=100 -> lower=0.0 upper=0.3 effort=50 velocity=100
